Commit message: Update

File: src/my_r2d2/urdf/r2d2.xacro (robot description, xacro)
@@ -8,4 +8,6 @@
   <xacro:property name="wheeldiam" value="0.07" />
   <xacro:property name="pi" value="3.1415" />
+  <xacro:property name="lens_length" value="0.04" />
+  <xacro:property name="lens_radius" value="0.02" />
   <material name="blue">
     <color rgba="0 0 0.8 1"/>
@@ -37,12 +39,19 @@
     <xacro:default_inertial mass="10"/>
   </link>
-    <link name="base_footprint">
-    </link>
-    <joint name="base_footprint_to_base_link" type="fixed">
-       <axis rpy="0 0 0" xyz="0 1 0"/>
-      <parent link="base_link"/>
-      <child link="base_footprint"/>
-      <origin rpy="0 0 0" xyz="0.0 0.0 -0.47"/>
-    </joint>
+  <link name = "lens">
+      <visual>
+        <origin xyz="0 0 0" rpy="0 0 0" />
+        <geometry>
+          <cylinder radius="${lens_radius}" length="${lens_length}"/>
+        </geometry>
+        <material name="black"/>
+      </visual>
+      <collision>
+        <origin xyz="0 0 0" rpy="-1.57 0 0" />
+        <geometry>
+          <cylinder radius="0.1" length="0.1"/>
+        </geometry>
+      </collision>
+</link>
   <xacro:macro name="wheel" params="prefix suffix reflect">
     <link name="${prefix}_${suffix}_wheel">
@@ -115,4 +124,6 @@
   <xacro:leg prefix="right" reflect="-1" />
   <xacro:leg prefix="left" reflect="1" />
+ <link name="base_footprint">
+    </link>
   <joint name="gripper_extension" type="prismatic">
     <parent link="base_link"/>
@@ -221,3 +232,14 @@
     <origin xyz="${.707*width+0.04} 0 ${.707*width}"/>
   </joint>
+ <joint name="tolens" type="fixed">
+    <parent link="box"/>
+    <child link="lens"/>
+    <origin xyz=" ${lens_length/2} 0 0" rpy= "0 ${-pi/2} 0"/>
+  </joint>
+    <joint name="base_footprint_to_base_link" type="fixed">
+       <axis rpy="0 0 0" xyz="0 1 0"/>
+      <parent link="base_link"/>
+      <child link="base_footprint"/>
+      <origin rpy="0 0 0" xyz="0.0 0.0 -0.47"/>
+    </joint>
 </robot>
